File: src/just-another-keyboard.kicad_sch (KiCad schematic)
At the start: 0 parts

Commit message: Start working on it
Parts:
- added U1: RP2040, Package_DFN_QFN:QFN-56-1EP_7x7mm_P0.4mm_EP3.2x3.2mm, symbol MCU_RaspberryPi:RP2040
Connections:
- new net: U1.1 (IOVDD), U1.10 (IOVDD), U1.22 (IOVDD), U1.33 (IOVDD), U1.42 (IOVDD), U1.49 (IOVDD)
- new net: U1.23 (DVDD), U1.50 (DVDD)
Changed lines of the file:
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@@
 	(generator_version "9.0")
 	(paper "A4")
+	(symbol
+		(lib_id "MCU_RaspberryPi:RP2040")
+		(at 73.66 111.76 0)
+		(unit 1)
+		(exclude_from_sim no)
+		(in_bom yes)
+		(on_board yes)
+		(dnp no)
+		(fields_autoplaced yes)
+		(property "Reference" "U1"
+			(at 75.8033 156.21 0)
+			(effects
+				(font
+					(size 1.27 1.27)
+				)
+				(justify left)
+			)
+		)
+		(property "Value" "RP2040"
+			(at 75.8033 158.75 0)
+			(effects
+				(font
+					(size 1.27 1.27)
+				)
+				(justify left)
+			)
+		)
+		(property "Footprint" "Package_DFN_QFN:QFN-56-1EP_7x7mm_P0.4mm_EP3.2x3.2mm"
+			(at 73.66 111.76 0)
+			(effects
+				(font
+					(size 1.27 1.27)
+				)
+				(hide yes)
+			)
+		)
+		(property "Datasheet" "https://datasheets.raspberrypi.com/rp2040/rp2040-datasheet.pdf"
+			(at 73.66 111.76 0)
+			(effects
+				(font
+					(size 1.27 1.27)
+				)
+				(hide yes)
+			)
+		)
+		(property "Description" "A microcontroller by Raspberry Pi"
+			(at 73.66 111.76 0)
+			(effects
+				(font
+					(size 1.27 1.27)
+				)
+				(hide yes)
+			)
+		)
+		(pin "24"
+		)
+		(pin "2"
+		)
+		(pin "16"
+		)
+		(pin "13"
+		)
+		(pin "44"
+		)
+		(pin "30"
+		)
+		(pin "21"
+		)
+		(pin "43"
+		)
+		(pin "17"
+		)
+		(pin "29"
+		)
+		(pin "49"
+		)
+		(pin "57"
+		)
+		(pin "27"
+		)
+		(pin "37"
+		)
+		(pin "42"
+		)
+		(pin "28"
+		)
+		(pin "41"
+		)
+		(pin "10"
+		)
+		(pin "55"
+		)
+		(pin "1"
+		)
+		(pin "40"
+		)
+		(pin "48"
+		)
+		(pin "22"
+		)
+		(pin "18"
+		)
+		(pin "53"
+		)
+		(pin "56"
+		)
+		(pin "19"
+		)
+		(pin "45"
+		)
+		(pin "6"
+		)
+		(pin "39"
+		)
+		(pin "25"
+		)
+		(pin "3"
+		)
+		(pin "46"
+		)
+		(pin "47"
+		)
+		(pin "20"
+		)
+		(pin "8"
+		)
+		(pin "4"
+		)
+		(pin "31"
+		)
+		(pin "34"
+		)
+		(pin "38"
+		)
+		(pin "26"
+		)
+		(pin "32"
+		)
+		(pin "54"
+		)
+		(pin "35"
+		)
+		(pin "51"
+		)
+		(pin "36"
+		)
+		(pin "7"
+		)
+		(pin "15"
+		)
+		(pin "33"
+		)
+		(pin "14"
+		)
+		(pin "50"
+		)
+		(pin "12"
+		)
+		(pin "11"
+		)
+		(pin "9"
+		)
+		(pin "5"
+		)
+		(pin "23"
+		)
+		(pin "52"
+		)
+		(instances
+			(project ""
+				(path "/58b2bf00-85ee-4776-bb6e-358369f1eff9"
+					(reference "U1")
+					(unit 1)
+				)
+			)
+		)
+	)
 	(sheet_instances
 		(path "/"
